File: isolated_input.kicad_sch (KiCad schematic)
At the start: 17 parts, among them Q1 PMV213SN, Q2 DMP610DL, Q3 2N7002, Q4 2N7002, U1 EL3H7, U2 AL5809, U4 EL3H7, U9 AL5809

Commit message: Get board name and version from text variable
Other:
- title: (none) -> ${BoardName}
Changed lines of the file:
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@@
 	(generator_version "8.99")
 	(paper "A4")
+	(title_block
+		(title "${BoardName}")
+		(date "2024-11-11")
+		(rev "${Version}")
+	)
 	(rectangle
 		(start 208.28 88.9)
