File: multi_input_edgy.kicad_sch (KiCad schematic)
At the start: 10 parts, among them J1 002, J2 002, J7 6V-24V, U18 SN74LVC1G125

Commit message: Get board name and version from text variable
Other:
- title: (none) -> ${BoardName}
Changed lines of the file:
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@@
 	(generator_version "8.99")
 	(paper "A4")
+	(title_block
+		(title "${BoardName}")
+		(date "2024-11-11")
+		(rev "${Version}")
+	)
 	(rectangle
 		(start 109.728 107.95)
